Commit message: Reset current baseline for robotarm_mt4
Document why the baseline reset was needed: repository rename, too many daily notes, and mixed student/hardware responsibilities. Set README and docs/CURRENT_BASELINE.md as the daily source of truth for the Mirobot/MT4 asset and hardware-transfer work.

File: assets/urdf/wlkata_mt4_official/wlkata_mt4_official.urdf (robot description, URDF)
Before this commit: robot wlkata_mt4_description, 12 links, 11 joints
Links:
- link base_link: geometry collision mesh filename=/home/spark-robotics/work/robotarm/robotarm_mt4/assets/urdf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; visual mesh filename=/home/spark-robotics/work/robotarm/robotarm_mt4/assets/urdf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
- link link1: geometry collision mesh filename=/home/spark-robotics/work/robotarm/robotarm_mt4/assets/urdf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; visual mesh filename=/home/spark-robotics/work/robotarm/robotarm_mt4/assets/urdf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
- link link10: geometry collision mesh filename=/home/spark-robotics/work/robotarm/robotarm_mt4/assets/urdf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; visual mesh filename=/home/spark-robotics/work/robotarm/robotarm_mt4/assets/urdf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
- link link11: geometry collision mesh filename=/home/spark-robotics/work/robotarm/robotarm_mt4/assets/urdf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; visual mesh filename=/home/spark-robotics/work/robotarm/robotarm_mt4/assets/urdf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
- link link2: geometry collision mesh filename=/home/spark-robotics/work/robotarm/robotarm_mt4/assets/urdf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; visual mesh filename=/home/spark-robotics/work/robotarm/robotarm_mt4/assets/urdf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
- link link3: geometry collision mesh filename=/home/spark-robotics/work/robotarm/robotarm_mt4/assets/urdf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; visual mesh filename=/home/spark-robotics/work/robotarm/robotarm_mt4/assets/urdf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
- link link4: geometry collision mesh filename=/home/spark-robotics/work/robotarm/robotarm_mt4/assets/urdf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; visual mesh filename=/home/spark-robotics/work/robotarm/robotarm_mt4/assets/urdf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
- link link5: geometry collision mesh filename=/home/spark-robotics/work/robotarm/robotarm_mt4/assets/urdf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; visual mesh filename=/home/spark-robotics/work/robotarm/robotarm_mt4/assets/urdf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
- link link6: geometry collision mesh filename=/home/spark-robotics/work/robotarm/robotarm_mt4/assets/urdf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; visual mesh filename=/home/spark-robotics/work/robotarm/robotarm_mt4/assets/urdf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
- link link7: geometry collision mesh filename=/home/spark-robotics/work/robotarm/robotarm_mt4/assets/urdf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; visual mesh filename=/home/spark-robotics/work/robotarm/robotarm_mt4/assets/urdf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
- link link8: geometry collision mesh filename=/home/spark-robotics/work/robotarm/robotarm_mt4/assets/urdf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; visual mesh filename=/home/spark-robotics/work/robotarm/robotarm_mt4/assets/urdf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
- link link9: geometry collision mesh filename=/home/spark-robotics/work/robotarm/robotarm_mt4/assets/urdf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; visual mesh filename=/home/spark-robotics/work/robotarm/robotarm_mt4/assets/urdf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
